File: pcbs/3x5_2/busterswoop/busterswoop.kicad_sch (KiCad schematic)
At the start: 42 parts, among them J1 TRRS, SW1 Choc, SW10 Choc, SW11 Choc, SW12 Choc, SW13 Choc, SW14 Choc, SW15 Choc, SW16 Choc, SW17 Choc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

Commit message: added new stls and images
Parts:
- RSW1: footprint arkenswoop:Reset -> Button_Switch_SMD:Panasonic_EVQPUJ_EVQPUA
Changed lines of the file:
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@@
       (effects (font (size 1.27 1.27)))
     )
-    (property "Footprint" "arkenswoop:Reset" (at 38.1 70.6119 0)
+    (property "Footprint" "Button_Switch_SMD:Panasonic_EVQPUJ_EVQPUA" (at 38.1 70.6119 0)
       (effects (font (size 1.27 1.27)) hide)
     )
